Commit message: creaded a working quadruped and a test controller

File: src/mechdog_gazebo/urdf/mechdog.urdf.xacro (robot description, xacro)
@@ -1,60 +1,315 @@
 <?xml version="1.0"?>
-<robot xmlns:xacro="http://www.ros.org/wiki/xacro" name="mechdog">
-  <!-- Simple colors -->
-  <material name="black"><color rgba="0 0 0 1"/></material>
-  <material name="gray"><color rgba="0.6 0.6 0.6 1"/></material>
-  <!-- Base -->
-  <link name="base_link">
-    <visual>
-      <origin xyz="0 0 0.15" rpy="0 0 0"/>
-      <geometry>
-        <box size="0.35 0.18 0.10"/>
-      </geometry>
-      <material name="gray"/>
-    </visual>
-    <collision>
-      <origin xyz="0 0 0.15" rpy="0 0 0"/>
-      <geometry>
-        <box size="0.35 0.18 0.10"/>
-      </geometry>
-    </collision>
+<!--
+  Quadrupedal Robot URDF/Xacro Model
+  Inspired by robots like HiWonder MechDog / Puppy
+  12 DOF: 3 joints per leg (hip_roll, hip_pitch, knee_pitch) x 4 legs
+  Leg naming convention:
+    FL = Front Left
+    FR = Front Right
+    RL = Rear Left
+    RR = Rear Right
+-->
+<robot name="quadruped" xmlns:xacro="http://www.ros.org/wiki/xacro">
+  <!-- ===================== PROPERTIES ===================== -->
+  <!-- Body dimensions -->
+  <xacro:property name="body_length" value="0.25"/>
+  <xacro:property name="body_width"  value="0.12"/>
+  <xacro:property name="body_height" value="0.055"/>
+  <xacro:property name="body_mass"   value="1.2"/>
+  <!-- Hip offset from body center -->
+  <xacro:property name="hip_x_offset" value="0.10"/>
+  <xacro:property name="hip_y_offset" value="0.065"/>
+  <xacro:property name="hip_z_offset" value="0.0"/>
+  <!-- Hip link dimensions -->
+  <xacro:property name="hip_length" value="0.04"/>
+  <xacro:property name="hip_radius" value="0.018"/>
+  <xacro:property name="hip_mass"   value="0.08"/>
+  <!-- Thigh link dimensions -->
+  <xacro:property name="thigh_length" value="0.085"/>
+  <xacro:property name="thigh_radius" value="0.014"/>
+  <xacro:property name="thigh_mass"   value="0.10"/>
+  <!-- Calf (shin) link dimensions -->
+  <xacro:property name="calf_length" value="0.095"/>
+  <xacro:property name="calf_radius" value="0.012"/>
+  <xacro:property name="calf_mass"   value="0.06"/>
+  <!-- Foot sphere -->
+  <xacro:property name="foot_radius" value="0.015"/>
+  <xacro:property name="foot_mass"   value="0.02"/>
+  <!-- Joint limits (radians) -->
+  <xacro:property name="hip_roll_min"  value="-0.6"/>
+  <xacro:property name="hip_roll_max"  value="0.6"/>
+  <xacro:property name="hip_pitch_min" value="-1.2"/>
+  <xacro:property name="hip_pitch_max" value="1.2"/>
+  <xacro:property name="knee_min"      value="-2.5"/>
+  <xacro:property name="knee_max"      value="-0.3"/>
+  <!-- Joint effort / velocity limits -->
+  <xacro:property name="joint_effort"   value="15.0"/>
+  <xacro:property name="joint_velocity" value="10.0"/>
+  <!-- Colors -->
+  <material name="dark_grey">
+    <color rgba="0.2 0.2 0.2 1.0"/>
+  </material>
+  <material name="light_grey">
+    <color rgba="0.6 0.6 0.6 1.0"/>
+  </material>
+  <material name="orange">
+    <color rgba="1.0 0.5 0.0 1.0"/>
+  </material>
+  <material name="black">
+    <color rgba="0.05 0.05 0.05 1.0"/>
+  </material>
+  <!-- ===================== INERTIA MACROS ===================== -->
+  <xacro:macro name="box_inertia" params="m x y z">
     <inertial>
-      <origin xyz="0 0 0.15" rpy="0 0 0"/>
-      <mass value="4.0"/>
-      <inertia ixx="0.05" ixy="0.0" ixz="0.0" iyy="0.10" iyz="0.0" izz="0.12"/>
+      <mass value="${m}"/>
+      <inertia ixx="${m*(y*y+z*z)/12}" ixy="0" ixz="0"
+               iyy="${m*(x*x+z*z)/12}" iyz="0"
+               izz="${m*(x*x+y*y)/12}"/>
     </inertial>
-  </link>
-  <!-- Four simple legs (fixed joints for now) -->
-  <xacro:macro name="leg" params="prefix x y">
-    <link name="${prefix}_link">
+  </xacro:macro>
+  <xacro:macro name="cylinder_inertia" params="m r l">
+    <inertial>
+      <mass value="${m}"/>
+      <inertia ixx="${m*(3*r*r+l*l)/12}" ixy="0" ixz="0"
+               iyy="${m*(3*r*r+l*l)/12}" iyz="0"
+               izz="${m*r*r/2}"/>
+    </inertial>
+  </xacro:macro>
+  <xacro:macro name="sphere_inertia" params="m r">
+    <inertial>
+      <mass value="${m}"/>
+      <inertia ixx="${2*m*r*r/5}" ixy="0" ixz="0"
+               iyy="${2*m*r*r/5}" iyz="0"
+               izz="${2*m*r*r/5}"/>
+    </inertial>
+  </xacro:macro>
+  <!-- ===================== LEG MACRO ===================== -->
+  <!--
+    Params:
+      prefix   : FL | FR | RL | RR
+      x_sign   : +1 (front) | -1 (rear)
+      y_sign   : +1 (left)  | -1 (right)
+  -->
+  <xacro:macro name="leg" params="prefix x_sign y_sign">
+    <!-- ── HIP ROLL JOINT ── -->
+    <joint name="${prefix}_hip_roll_joint" type="revolute">
+      <parent link="base_link"/>
+      <child  link="${prefix}_hip_link"/>
+      <origin xyz="${x_sign*hip_x_offset} ${y_sign*hip_y_offset} ${hip_z_offset}" rpy="0 0 0"/>
+      <axis xyz="1 0 0"/>
+      <limit lower="${hip_roll_min}" upper="${hip_roll_max}"
+             effort="${joint_effort}" velocity="${joint_velocity}"/>
+      <dynamics damping="0.1" friction="0.05"/>
+    </joint>
+    <link name="${prefix}_hip_link">
+      <xacro:cylinder_inertia m="${hip_mass}" r="${hip_radius}" l="${hip_length}"/>
       <visual>
-        <origin xyz="${x} ${y} 0.08" rpy="0 0 0"/>
-        <geometry>
-          <cylinder radius="0.02" length="0.16"/>
+        <origin xyz="0 ${y_sign*hip_length/2} 0" rpy="${pi/2} 0 0"/>
+        <geometry>
+          <cylinder radius="${hip_radius}" length="${hip_length}"/>
+        </geometry>
+        <material name="orange"/>
+      </visual>
+      <collision>
+        <origin xyz="0 ${y_sign*hip_length/2} 0" rpy="${pi/2} 0 0"/>
+        <geometry>
+          <cylinder radius="${hip_radius}" length="${hip_length}"/>
+        </geometry>
+      </collision>
+    </link>
+    <!-- ── HIP PITCH JOINT ── -->
+    <joint name="${prefix}_hip_pitch_joint" type="revolute">
+      <parent link="${prefix}_hip_link"/>
+      <child  link="${prefix}_thigh_link"/>
+      <origin xyz="0 ${y_sign*hip_length} 0" rpy="0 0 0"/>
+      <axis xyz="0 1 0"/>
+      <limit lower="${hip_pitch_min}" upper="${hip_pitch_max}"
+             effort="${joint_effort}" velocity="${joint_velocity}"/>
+      <dynamics damping="0.1" friction="0.05"/>
+    </joint>
+    <link name="${prefix}_thigh_link">
+      <xacro:cylinder_inertia m="${thigh_mass}" r="${thigh_radius}" l="${thigh_length}"/>
+      <visual>
+        <origin xyz="0 0 ${-thigh_length/2}" rpy="0 0 0"/>
+        <geometry>
+          <cylinder radius="${thigh_radius}" length="${thigh_length}"/>
+        </geometry>
+        <material name="light_grey"/>
+      </visual>
+      <collision>
+        <origin xyz="0 0 ${-thigh_length/2}" rpy="0 0 0"/>
+        <geometry>
+          <cylinder radius="${thigh_radius}" length="${thigh_length}"/>
+        </geometry>
+      </collision>
+    </link>
+    <!-- ── KNEE PITCH JOINT ── -->
+    <joint name="${prefix}_knee_joint" type="revolute">
+      <parent link="${prefix}_thigh_link"/>
+      <child  link="${prefix}_calf_link"/>
+      <origin xyz="0 0 ${-thigh_length}" rpy="0 0 0"/>
+      <axis xyz="0 1 0"/>
+      <limit lower="${knee_min}" upper="${knee_max}"
+             effort="${joint_effort}" velocity="${joint_velocity}"/>
+      <dynamics damping="0.1" friction="0.05"/>
+    </joint>
+    <link name="${prefix}_calf_link">
+      <xacro:cylinder_inertia m="${calf_mass}" r="${calf_radius}" l="${calf_length}"/>
+      <visual>
+        <origin xyz="0 0 ${-calf_length/2}" rpy="0 0 0"/>
+        <geometry>
+          <cylinder radius="${calf_radius}" length="${calf_length}"/>
+        </geometry>
+        <material name="dark_grey"/>
+      </visual>
+      <collision>
+        <origin xyz="0 0 ${-calf_length/2}" rpy="0 0 0"/>
+        <geometry>
+          <cylinder radius="${calf_radius}" length="${calf_length}"/>
+        </geometry>
+      </collision>
+    </link>
+    <!-- ── FOOT (fixed) ── -->
+    <joint name="${prefix}_foot_joint" type="fixed">
+      <parent link="${prefix}_calf_link"/>
+      <child  link="${prefix}_foot_link"/>
+      <origin xyz="0 0 ${-calf_length}" rpy="0 0 0"/>
+    </joint>
+    <link name="${prefix}_foot_link">
+      <xacro:sphere_inertia m="${foot_mass}" r="${foot_radius}"/>
+      <visual>
+        <origin xyz="0 0 0" rpy="0 0 0"/>
+        <geometry>
+          <sphere radius="${foot_radius}"/>
         </geometry>
         <material name="black"/>
       </visual>
       <collision>
-        <origin xyz="${x} ${y} 0.08" rpy="0 0 0"/>
-        <geometry>
-          <cylinder radius="0.02" length="0.16"/>
-        </geometry>
+        <origin xyz="0 0 0" rpy="0 0 0"/>
+        <geometry>
+          <sphere radius="${foot_radius}"/>
+        </geometry>
+        <contact_coefficients mu="0.8" kp="1000000.0" kd="100.0"/>
       </collision>
-      <inertial>
-        <origin xyz="${x} ${y} 0.08" rpy="0 0 0"/>
-        <mass value="0.2"/>
-        <inertia ixx="0.0002" ixy="0.0" ixz="0.0" iyy="0.0002" iyz="0.0" izz="0.0002"/>
-      </inertial>
     </link>
-    <joint name="${prefix}_joint" type="fixed">
-      <parent link="base_link"/>
-      <child link="${prefix}_link"/>
+  </xacro:macro>
+  <!-- ===================== BASE LINK ===================== -->
+  <link name="base_link">
+    <xacro:box_inertia m="${body_mass}" x="${body_length}" y="${body_width}" z="${body_height}"/>
+    <visual>
       <origin xyz="0 0 0" rpy="0 0 0"/>
-    </joint>
-  </xacro:macro>
-  <!-- front-left, front-right, rear-left, rear-right -->
-  <xacro:leg prefix="fl" x="0.13"  y="0.08"/>
-  <xacro:leg prefix="fr" x="0.13"  y="-0.08"/>
-  <xacro:leg prefix="rl" x="-0.13" y="0.08"/>
-  <xacro:leg prefix="rr" x="-0.13" y="-0.08"/>
+      <geometry>
+        <box size="${body_length} ${body_width} ${body_height}"/>
+      </geometry>
+      <material name="dark_grey"/>
+    </visual>
+    <collision>
+      <origin xyz="0 0 0" rpy="0 0 0"/>
+      <geometry>
+        <box size="${body_length} ${body_width} ${body_height}"/>
+      </geometry>
+    </collision>
+  </link>
+  <!-- IMU link (center of body) -->
+  <joint name="imu_joint" type="fixed">
+    <parent link="base_link"/>
+    <child  link="imu_link"/>
+    <origin xyz="0 0 0" rpy="0 0 0"/>
+  </joint>
+  <link name="imu_link"/>
+  <!-- Camera link (front face) -->
+  <joint name="camera_joint" type="fixed">
+    <parent link="base_link"/>
+    <child  link="camera_link"/>
+    <origin xyz="${body_length/2} 0 ${body_height/4}" rpy="0 0 0"/>
+  </joint>
+  <link name="camera_link">
+    <visual>
+      <geometry>
+        <box size="0.015 0.06 0.015"/>
+      </geometry>
+      <material name="black"/>
+    </visual>
+  </link>
+  <!-- ===================== INSTANTIATE LEGS ===================== -->
+  <xacro:leg prefix="FL" x_sign="1"  y_sign="1"/>
+  <xacro:leg prefix="FR" x_sign="1"  y_sign="-1"/>
+  <xacro:leg prefix="RL" x_sign="-1" y_sign="1"/>
+  <xacro:leg prefix="RR" x_sign="-1" y_sign="-1"/>
+  <!-- ===================== GAZEBO PLUGINS ===================== -->
+  <!-- Gazebo contact sensors for feet -->
+  <xacro:macro name="foot_contact_sensor" params="prefix">
+    <gazebo reference="${prefix}_foot_link">
+      <sensor name="${prefix}_foot_contact" type="contact">
+        <contact>
+          <collision>${prefix}_foot_link_collision</collision>
+        </contact>
+        <update_rate>100</update_rate>
+        <plugin name="${prefix}_foot_contact_plugin" filename="libgazebo_ros_bumper.so">
+          <bumperTopicName>${prefix}_foot_contact</bumperTopicName>
+          <frameName>${prefix}_foot_link</frameName>
+        </plugin>
+      </sensor>
+      <material>Gazebo/Black</material>
+    </gazebo>
+  </xacro:macro>
+  <xacro:foot_contact_sensor prefix="FL"/>
+  <xacro:foot_contact_sensor prefix="FR"/>
+  <xacro:foot_contact_sensor prefix="RL"/>
+  <xacro:foot_contact_sensor prefix="RR"/>
+  <!-- IMU Sensor -->
+  <gazebo reference="imu_link">
+    <sensor name="imu_sensor" type="imu">
+      <always_on>true</always_on>
+      <update_rate>200</update_rate>
+      <visualize>false</visualize>
+      <plugin name="imu_plugin" filename="libgazebo_ros_imu_sensor.so">
+        <topicName>imu/data</topicName>
+        <bodyName>imu_link</bodyName>
+        <updateRateHZ>200.0</updateRateHZ>
+        <gaussianNoise>0.0</gaussianNoise>
+        <xyzOffset>0 0 0</xyzOffset>
+        <rpyOffset>0 0 0</rpyOffset>
+        <frameName>imu_link</frameName>
+        <initialOrientationAsReference>false</initialOrientationAsReference>
+      </plugin>
+    </sensor>
+  </gazebo>
+  <!-- Camera -->
+  <gazebo reference="camera_link">
+    <sensor type="camera" name="front_camera">
+      <update_rate>30.0</update_rate>
+      <camera name="head">
+        <horizontal_fov>1.3962634</horizontal_fov>
+        <image>
+          <width>640</width>
+          <height>480</height>
+          <format>R8G8B8</format>
+        </image>
+        <clip>
+          <near>0.02</near>
+          <far>300</far>
+        </clip>
+      </camera>
+      <plugin name="camera_controller" filename="libgazebo_ros_camera.so">
+        <alwaysOn>true</alwaysOn>
+        <updateRate>30.0</updateRate>
+        <cameraName>front_camera</cameraName>
+        <imageTopicName>image_raw</imageTopicName>
+        <cameraInfoTopicName>camera_info</cameraInfoTopicName>
+        <frameName>camera_link</frameName>
+      </plugin>
+    </sensor>
+    <material>Gazebo/Black</material>
+  </gazebo>
+  <!-- ROS 2 Control Plugin -->
+  <gazebo>
+    <plugin filename="libgazebo_ros2_control.so" name="gazebo_ros2_control">
+      <parameters>$(find mechdog_gazebo)/config/ros2_control.yaml</parameters>
+    </plugin>
+  </gazebo>
+  <!-- Body material -->
+  <gazebo reference="base_link">
+    <material>Gazebo/DarkGrey</material>
+  </gazebo>
 </robot>
