Commit message: solved orb-slam3 build errors and integrated monodepth with dept image to pointcloud module

File: src/quadruped_gazebo/urdf/quadruped.urdf.xacro (robot description, xacro)
@@ -232,4 +232,11 @@
     </visual>
   </link>
+  <!-- Camera optical link (rotated to ROS standard: Z-forward, X-right, Y-down) -->
+  <joint name="camera_optical_joint" type="fixed">
+    <parent link="camera_link"/>
+    <child  link="camera_link_optical"/>
+    <origin xyz="0 0 0" rpy="${-pi/2} 0 ${-pi/2}"/>
+  </joint>
+  <link name="camera_link_optical"/>
   <!-- ===================== INSTANTIATE LEGS ===================== -->
   <xacro:leg prefix="FL" x_sign="1"  y_sign="1"/>
@@ -326,5 +333,5 @@
       <update_rate>30</update_rate>
       <topic>front_camera/image_raw</topic>
-      <gz_frame_id>camera_link</gz_frame_id>
+      <gz_frame_id>camera_link_optical</gz_frame_id>
       <camera>
         <horizontal_fov>1.3962634</horizontal_fov>
