Commit message: feat(quadruped_kinematics): Spot Micro geometry as a shared package
Leg IK/FK lived in two copies — the gait controller's node and the leg
odometry's kinematics module — with hand-transcribed link lengths that
could drift from the URDF and from each other. Extract closed-form leg
IK/FK/Jacobian and whole-body IK into quadruped_kinematics (pure numpy),
and have both consumers import it. Its tests parse the URDF xacro, so a
geometry change in one place now fails the build rather than silently
disagreeing.

The URDF moves to real Spot Micro geometry (0.186 x 0.078 m hip pivots,
55 mm hip link, 107.5/130 mm leg links) and derives the stand pose from
stand_height so the robot spawns standing.

The gait itself is rewritten around a pure-python gait.py: Bezier-swing
with per-leg stride vectors (v + w x r, so yaw produces tangential
strides), trot and walk from GAIT_LIBRARY, tuning via ROS parameters in
config/gait_params.yaml. A zero command finishes the cycle before
standing. Validated headless: 0.2-0.3 m/s straight with <2 deg roll and
pitch. The old duty-0.5 flight trot falls under position control; the
gait_demo scripts that drove it are removed.

Co-Authored-By: Claude Opus 5 <noreply@anthropic.com>

File: src/quadruped_gazebo/urdf/quadruped.urdf.xacro (robot description, xacro)
@@ -1,65 +1,97 @@
 <?xml version="1.0"?>
 <!--
-  Quadrupedal Robot URDF/Xacro Model
-  Inspired by robots like HiWonder MechDog / Puppy
-  12 DOF: 3 joints per leg (hip_roll, hip_pitch, knee_pitch) x 4 legs
-  Leg naming convention:
-    FL = Front Left
-    FR = Front Right
-    RL = Rear Left
-    RR = Rear Right
+  Spot Micro quadruped — URDF/Xacro model for Gazebo Harmonic.
+  Geometry follows the open-source Spot Micro (KDY0532 / mike4192 spotMicro):
+    0.186 m between front and rear hip pivots, 0.078 m between left and right,
+    0.055 m abduction ("shoulder") link, 0.1075 m upper leg, 0.130 m lower leg.
+  12 DOF: hip_roll (abduction), hip_pitch, knee per leg. All four knees point
+  backward (Spot configuration): the upper leg angles back from the hip and
+  the lower leg folds forward under the body, so the knee angle is always
+  negative.
+  Leg naming: FL / FR / RL / RR (front/rear, left/right).
+  The link lengths here are mirrored in python by
+  src/quadruped_kinematics/quadruped_kinematics/geometry.py; a unit test in
+  that package parses this file and fails if the two disagree. Change the
+  geometry in both places or not at all.
 -->
 <robot name="quadruped" xmlns:xacro="http://www.ros.org/wiki/xacro">
-  <!-- ===================== PROPERTIES ===================== -->
-  <!-- Body dimensions -->
-  <xacro:property name="body_length" value="0.25"/>
-  <xacro:property name="body_width"  value="0.12"/>
-  <xacro:property name="body_height" value="0.055"/>
-  <xacro:property name="body_mass"   value="1.2"/>
-  <!-- Hip offset from body center -->
-  <xacro:property name="hip_x_offset" value="0.10"/>
-  <xacro:property name="hip_y_offset" value="0.065"/>
-  <xacro:property name="hip_z_offset" value="0.0"/>
-  <!-- Hip link dimensions -->
-  <xacro:property name="hip_length" value="0.04"/>
-  <xacro:property name="hip_radius" value="0.018"/>
-  <xacro:property name="hip_mass"   value="0.08"/>
-  <!-- Thigh link dimensions -->
-  <xacro:property name="thigh_length" value="0.085"/>
-  <xacro:property name="thigh_radius" value="0.014"/>
-  <xacro:property name="thigh_mass"   value="0.10"/>
-  <!-- Calf (shin) link dimensions -->
-  <xacro:property name="calf_length" value="0.095"/>
-  <xacro:property name="calf_radius" value="0.012"/>
-  <xacro:property name="calf_mass"   value="0.06"/>
-  <!-- Foot sphere -->
+  <!-- ===================== GEOMETRY (metres, kg) ===================== -->
+  <!-- Leg kinematic parameters — keep in sync with quadruped_kinematics -->
+  <xacro:property name="hip_x"       value="0.093"/>   <!-- half the hip-to-hip length -->
+  <xacro:property name="hip_y"       value="0.039"/>   <!-- half the hip-to-hip width -->
+  <xacro:property name="hip_link"    value="0.055"/>   <!-- abduction link, pivot to leg plane -->
+  <xacro:property name="upper_leg"   value="0.1075"/>
+  <xacro:property name="lower_leg"   value="0.130"/>
   <xacro:property name="foot_radius" value="0.015"/>
+  <!-- Nominal stand: base_link height above ground. The gait controller's
+       body_height parameter defaults to the same value; ros2_control
+       initial_value is derived from it below so the robot spawns standing. -->
+  <xacro:property name="stand_height" value="0.16"/>
+  <!-- Body shell (main chassis + head + tail), all one rigid link -->
+  <xacro:property name="body_length" value="0.20"/>
+  <xacro:property name="body_width"  value="0.09"/>
+  <xacro:property name="body_height" value="0.06"/>
+  <xacro:property name="head_length" value="0.07"/>
+  <xacro:property name="head_width"  value="0.08"/>
+  <xacro:property name="head_height" value="0.05"/>
+  <xacro:property name="tail_length" value="0.05"/>
+  <xacro:property name="body_mass"   value="1.30"/>
+  <!-- Leg link visuals/masses. Hip and upper leg each house a servo. -->
+  <xacro:property name="hip_box_x"  value="0.060"/>
+  <xacro:property name="hip_box_z"  value="0.045"/>
+  <xacro:property name="hip_mass"   value="0.15"/>
+  <xacro:property name="upper_box_x" value="0.030"/>
+  <xacro:property name="upper_box_y" value="0.025"/>
+  <xacro:property name="upper_mass"  value="0.16"/>
+  <xacro:property name="lower_box_x" value="0.020"/>
+  <xacro:property name="lower_box_y" value="0.015"/>
+  <xacro:property name="lower_mass"  value="0.05"/>
   <xacro:property name="foot_mass"   value="0.02"/>
-  <!-- Joint limits (radians) -->
-  <xacro:property name="hip_roll_min"  value="-0.6"/>
-  <xacro:property name="hip_roll_max"  value="0.6"/>
+  <!-- Joint limits (rad). Knee never passes through straight. -->
+  <xacro:property name="hip_roll_min"  value="-0.75"/>
+  <xacro:property name="hip_roll_max"  value="0.75"/>
   <xacro:property name="hip_pitch_min" value="-1.2"/>
-  <xacro:property name="hip_pitch_max" value="1.2"/>
-  <xacro:property name="knee_min"      value="-2.5"/>
-  <xacro:property name="knee_max"      value="-0.3"/>
-  <!-- Joint effort / velocity limits -->
-  <xacro:property name="joint_effort"   value="15.0"/>
-  <xacro:property name="joint_velocity" value="10.0"/>
+  <xacro:property name="hip_pitch_max" value="1.6"/>
+  <xacro:property name="knee_min"      value="-2.7"/>
+  <xacro:property name="knee_max"      value="-0.35"/>
+  <!-- 35 kg·cm class hobby servo: ~3.4 N·m stall, ~0.15 s / 60° -->
+  <xacro:property name="joint_effort"   value="3.4"/>
+  <xacro:property name="joint_velocity" value="7.0"/>
+  <xacro:property name="joint_damping"  value="0.02"/>
+  <xacro:property name="joint_friction" value="0.02"/>
+  <!-- Stand pose derived from the geometry: foot straight below the hip
+       pitch joint at reach h = stand_height - foot_radius (2-link IK). -->
+  <xacro:property name="stand_reach" value="${stand_height - foot_radius}"/>
+  <xacro:property name="stand_knee"
+    value="${-acos((stand_reach**2 - upper_leg**2 - lower_leg**2) / (2*upper_leg*lower_leg))}"/>
+  <xacro:property name="stand_hip_pitch"
+    value="${acos((upper_leg**2 + stand_reach**2 - lower_leg**2) / (2*upper_leg*stand_reach))}"/>
+  <!-- ICM-42688-P-class low-cost 6-axis IMU profile.
+       The white-noise values are the datasheet RMS figures for a 100 Hz
+       bandwidth (appropriate for the 200 Hz output rate below). Bias limits
+       are treated as 3-sigma turn-on errors. Gazebo's slow bias process is a
+       practical approximation because the real temperature history is not
+       simulated. All values use REP-103 SI units. -->
+  <xacro:property name="imu_update_rate" value="200.0"/>
+  <xacro:property name="imu_gyro_noise_stddev" value="0.0004886921906"/>
+  <xacro:property name="imu_gyro_bias_stddev" value="0.002908882087"/>
+  <xacro:property name="imu_gyro_dynamic_bias_stddev" value="0.0000872664626"/>
+  <xacro:property name="imu_gyro_dynamic_bias_correlation_time" value="300.0"/>
+  <xacro:property name="imu_gyro_precision" value="0.001065264436"/>
+  <xacro:property name="imu_accel_xy_noise_stddev" value="0.0063743225"/>
+  <xacro:property name="imu_accel_z_noise_stddev" value="0.006864655"/>
+  <xacro:property name="imu_accel_bias_stddev" value="0.06537766667"/>
+  <xacro:property name="imu_accel_dynamic_bias_stddev" value="0.004903325"/>
+  <xacro:property name="imu_accel_dynamic_bias_correlation_time" value="300.0"/>
+  <xacro:property name="imu_accel_precision" value="0.00478840332"/>
   <!-- Colors -->
-  <material name="dark_grey">
-    <color rgba="0.2 0.2 0.2 1.0"/>
-  </material>
-  <material name="light_grey">
-    <color rgba="0.6 0.6 0.6 1.0"/>
-  </material>
-  <material name="orange">
-    <color rgba="1.0 0.5 0.0 1.0"/>
-  </material>
-  <material name="black">
-    <color rgba="0.05 0.05 0.05 1.0"/>
-  </material>
+  <material name="yellow"><color rgba="0.95 0.75 0.10 1.0"/></material>
+  <material name="dark_grey"><color rgba="0.20 0.20 0.20 1.0"/></material>
+  <material name="light_grey"><color rgba="0.65 0.65 0.65 1.0"/></material>
+  <material name="black"><color rgba="0.05 0.05 0.05 1.0"/></material>
   <!-- ===================== INERTIA MACROS ===================== -->
-  <xacro:macro name="box_inertia" params="m x y z">
+  <xacro:macro name="box_inertial" params="m x y z *origin">
     <inertial>
+      <xacro:insert_block name="origin"/>
       <mass value="${m}"/>
       <inertia ixx="${m*(y*y+z*z)/12}" ixy="0" ixz="0"
@@ -68,13 +100,5 @@
     </inertial>
   </xacro:macro>
-  <xacro:macro name="cylinder_inertia" params="m r l">
-    <inertial>
-      <mass value="${m}"/>
-      <inertia ixx="${m*(3*r*r+l*l)/12}" ixy="0" ixz="0"
-               iyy="${m*(3*r*r+l*l)/12}" iyz="0"
-               izz="${m*r*r/2}"/>
-    </inertial>
-  </xacro:macro>
-  <xacro:macro name="sphere_inertia" params="m r">
+  <xacro:macro name="sphere_inertial" params="m r">
     <inertial>
       <mass value="${m}"/>
@@ -86,130 +110,157 @@
   <!-- ===================== LEG MACRO ===================== -->
   <!--
-    Params:
-      prefix   : FL | FR | RL | RR
-      x_sign   : +1 (front) | -1 (rear)
-      y_sign   : +1 (left)  | -1 (right)
+    prefix : FL | FR | RL | RR
+    x_sign : +1 front | -1 rear
+    y_sign : +1 left  | -1 right
   -->
   <xacro:macro name="leg" params="prefix x_sign y_sign">
-    <!-- ── HIP ROLL JOINT ── -->
+    <!-- HIP ROLL (abduction) — pivot on the body side -->
     <joint name="${prefix}_hip_roll_joint" type="revolute">
       <parent link="base_link"/>
       <child  link="${prefix}_hip_link"/>
-      <origin xyz="${x_sign*hip_x_offset} ${y_sign*hip_y_offset} ${hip_z_offset}" rpy="0 0 0"/>
+      <origin xyz="${x_sign*hip_x} ${y_sign*hip_y} 0" rpy="0 0 0"/>
       <axis xyz="1 0 0"/>
       <limit lower="${hip_roll_min}" upper="${hip_roll_max}"
              effort="${joint_effort}" velocity="${joint_velocity}"/>
-      <dynamics damping="0.1" friction="0.05"/>
+      <dynamics damping="${joint_damping}" friction="${joint_friction}"/>
     </joint>
+    <!-- Hip link: servo block carrying the leg plane outboard -->
     <link name="${prefix}_hip_link">
-      <xacro:cylinder_inertia m="${hip_mass}" r="${hip_radius}" l="${hip_length}"/>
+      <xacro:box_inertial m="${hip_mass}" x="${hip_box_x}" y="${hip_link}" z="${hip_box_z}">
+        <origin xyz="0 ${y_sign*hip_link/2} 0" rpy="0 0 0"/>
+      </xacro:box_inertial>
       <visual>
-        <origin xyz="0 ${y_sign*hip_length/2} 0" rpy="${pi/2} 0 0"/>
-        <geometry>
-          <cylinder radius="${hip_radius}" length="${hip_length}"/>
-        </geometry>
-        <material name="orange"/>
+        <origin xyz="0 ${y_sign*hip_link/2} 0" rpy="0 0 0"/>
+        <geometry><box size="${hip_box_x} ${hip_link} ${hip_box_z}"/></geometry>
+        <material name="dark_grey"/>
       </visual>
       <collision>
-        <origin xyz="0 ${y_sign*hip_length/2} 0" rpy="${pi/2} 0 0"/>
-        <geometry>
-          <cylinder radius="${hip_radius}" length="${hip_length}"/>
-        </geometry>
+        <origin xyz="0 ${y_sign*hip_link/2} 0" rpy="0 0 0"/>
+        <geometry><box size="${hip_box_x} ${hip_link} ${hip_box_z}"/></geometry>
       </collision>
     </link>
-    <!-- ── HIP PITCH JOINT ── -->
+    <!-- HIP PITCH — in the leg plane, outboard end of the hip link -->
     <joint name="${prefix}_hip_pitch_joint" type="revolute">
       <parent link="${prefix}_hip_link"/>
-      <child  link="${prefix}_thigh_link"/>
-      <origin xyz="0 ${y_sign*hip_length} 0" rpy="0 0 0"/>
+      <child  link="${prefix}_upper_leg_link"/>
+      <origin xyz="0 ${y_sign*hip_link} 0" rpy="0 0 0"/>
       <axis xyz="0 1 0"/>
       <limit lower="${hip_pitch_min}" upper="${hip_pitch_max}"
              effort="${joint_effort}" velocity="${joint_velocity}"/>
-      <dynamics damping="0.1" friction="0.05"/>
+      <dynamics damping="${joint_damping}" friction="${joint_friction}"/>
     </joint>
-    <link name="${prefix}_thigh_link">
-      <xacro:cylinder_inertia m="${thigh_mass}" r="${thigh_radius}" l="${thigh_length}"/>
+    <link name="${prefix}_upper_leg_link">
+      <xacro:box_inertial m="${upper_mass}" x="${upper_box_x}" y="${upper_box_y}" z="${upper_leg}">
+        <origin xyz="0 0 ${-upper_leg/2}" rpy="0 0 0"/>
+      </xacro:box_inertial>
       <visual>
-        <origin xyz="0 0 ${-thigh_length/2}" rpy="0 0 0"/>
-        <geometry>
-          <cylinder radius="${thigh_radius}" length="${thigh_length}"/>
-        </geometry>
+        <origin xyz="0 0 ${-upper_leg/2}" rpy="0 0 0"/>
+        <geometry><box size="${upper_box_x} ${upper_box_y} ${upper_leg}"/></geometry>
+        <material name="yellow"/>
+      </visual>
+      <collision>
+        <origin xyz="0 0 ${-upper_leg/2}" rpy="0 0 0"/>
+        <geometry><box size="${upper_box_x} ${upper_box_y} ${upper_leg}"/></geometry>
+      </collision>
+    </link>
+    <!-- KNEE -->
+    <joint name="${prefix}_knee_joint" type="revolute">
+      <parent link="${prefix}_upper_leg_link"/>
+      <child  link="${prefix}_lower_leg_link"/>
+      <origin xyz="0 0 ${-upper_leg}" rpy="0 0 0"/>
+      <axis xyz="0 1 0"/>
+      <limit lower="${knee_min}" upper="${knee_max}"
+             effort="${joint_effort}" velocity="${joint_velocity}"/>
+      <dynamics damping="${joint_damping}" friction="${joint_friction}"/>
+    </joint>
+    <link name="${prefix}_lower_leg_link">
+      <xacro:box_inertial m="${lower_mass}" x="${lower_box_x}" y="${lower_box_y}" z="${lower_leg}">
+        <origin xyz="0 0 ${-lower_leg/2}" rpy="0 0 0"/>
+      </xacro:box_inertial>
+      <visual>
+        <origin xyz="0 0 ${-lower_leg/2}" rpy="0 0 0"/>
+        <geometry><box size="${lower_box_x} ${lower_box_y} ${lower_leg}"/></geometry>
         <material name="light_grey"/>
       </visual>
       <collision>
-        <origin xyz="0 0 ${-thigh_length/2}" rpy="0 0 0"/>
-        <geometry>
-          <cylinder radius="${thigh_radius}" length="${thigh_length}"/>
-        </geometry>
+        <origin xyz="0 0 ${-lower_leg/2}" rpy="0 0 0"/>
+        <geometry><box size="${lower_box_x} ${lower_box_y} ${lower_leg}"/></geometry>
       </collision>
     </link>
-    <!-- ── KNEE PITCH JOINT ── -->
-    <joint name="${prefix}_knee_joint" type="revolute">
-      <parent link="${prefix}_thigh_link"/>
-      <child  link="${prefix}_calf_link"/>
-      <origin xyz="0 0 ${-thigh_length}" rpy="0 0 0"/>
-      <axis xyz="0 1 0"/>
-      <limit lower="${knee_min}" upper="${knee_max}"
-             effort="${joint_effort}" velocity="${joint_velocity}"/>
-      <dynamics damping="0.1" friction="0.05"/>
-    </joint>
-    <link name="${prefix}_calf_link">
-      <xacro:cylinder_inertia m="${calf_mass}" r="${calf_radius}" l="${calf_length}"/>
-      <visual>
-        <origin xyz="0 0 ${-calf_length/2}" rpy="0 0 0"/>
-        <geometry>
-          <cylinder radius="${calf_radius}" length="${calf_length}"/>
-        </geometry>
-        <material name="dark_grey"/>
-      </visual>
-      <collision>
-        <origin xyz="0 0 ${-calf_length/2}" rpy="0 0 0"/>
-        <geometry>
-          <cylinder radius="${calf_radius}" length="${calf_length}"/>
-        </geometry>
-      </collision>
-    </link>
-    <!-- ── FOOT (fixed) ── -->
+    <!-- FOOT (fixed rubber ball) -->
     <joint name="${prefix}_foot_joint" type="fixed">
-      <parent link="${prefix}_calf_link"/>
+      <parent link="${prefix}_lower_leg_link"/>
       <child  link="${prefix}_foot_link"/>
-      <origin xyz="0 0 ${-calf_length}" rpy="0 0 0"/>
+      <origin xyz="0 0 ${-lower_leg}" rpy="0 0 0"/>
     </joint>
     <link name="${prefix}_foot_link">
-      <xacro:sphere_inertia m="${foot_mass}" r="${foot_radius}"/>
+      <xacro:sphere_inertial m="${foot_mass}" r="${foot_radius}"/>
       <visual>
-        <origin xyz="0 0 0" rpy="0 0 0"/>
-        <geometry>
-          <sphere radius="${foot_radius}"/>
-        </geometry>
+        <geometry><sphere radius="${foot_radius}"/></geometry>
         <material name="black"/>
       </visual>
       <collision>
-        <origin xyz="0 0 0" rpy="0 0 0"/>
-        <geometry>
-          <sphere radius="${foot_radius}"/>
-        </geometry>
-        <contact_coefficients mu="0.8" kp="1000000.0" kd="100.0"/>
+        <geometry><sphere radius="${foot_radius}"/></geometry>
       </collision>
     </link>
-  </xacro:macro>
-  <!-- ===================== BASE LINK ===================== -->
+    <gazebo reference="${prefix}_foot_link">
+      <mu1>1.0</mu1>
+      <mu2>1.0</mu2>
+      <kp>1000000.0</kp>
+      <kd>100.0</kd>
+    </gazebo>
+    <!-- Foot contact sensor (gz-sim); available for contact-based stance
+         detection, not bridged to ROS by default. The URDF→SDF conversion
+         lumps the fixed foot link into the lower leg and renames its
+         collision, so the sensor must name the lumped collision. -->
+    <gazebo reference="${prefix}_lower_leg_link">
+      <sensor name="${prefix}_foot_contact" type="contact">
+        <always_on>true</always_on>
+        <update_rate>100</update_rate>
+        <topic>${prefix}_foot_contact</topic>
+        <contact>
+          <collision>${prefix}_lower_leg_link_fixed_joint_lump__${prefix}_foot_link_collision_1</collision>
+        </contact>
+      </sensor>
+    </gazebo>
+  </xacro:macro>
+  <!-- ===================== BODY ===================== -->
   <link name="base_link">
-    <xacro:box_inertia m="${body_mass}" x="${body_length}" y="${body_width}" z="${body_height}"/>
+    <xacro:box_inertial m="${body_mass}" x="${body_length + head_length}" y="${body_width}" z="${body_height}">
+      <origin xyz="0.01 0 0" rpy="0 0 0"/>
+    </xacro:box_inertial>
+    <!-- main chassis -->
     <visual>
-      <origin xyz="0 0 0" rpy="0 0 0"/>
-      <geometry>
-        <box size="${body_length} ${body_width} ${body_height}"/>
-      </geometry>
+      <geometry><box size="${body_length} ${body_width} ${body_height}"/></geometry>
+      <material name="yellow"/>
+    </visual>
+    <collision>
+      <geometry><box size="${body_length} ${body_width} ${body_height}"/></geometry>
+    </collision>
+    <!-- head -->
+    <visual>
+      <origin xyz="${body_length/2 + head_length/2} 0 ${(body_height - head_height)/2}" rpy="0 0 0"/>
+      <geometry><box size="${head_length} ${head_width} ${head_height}"/></geometry>
       <material name="dark_grey"/>
     </visual>
     <collision>
-      <origin xyz="0 0 0" rpy="0 0 0"/>
-      <geometry>
-        <box size="${body_length} ${body_width} ${body_height}"/>
-      </geometry>
+      <origin xyz="${body_length/2 + head_length/2} 0 ${(body_height - head_height)/2}" rpy="0 0 0"/>
+      <geometry><box size="${head_length} ${head_width} ${head_height}"/></geometry>
     </collision>
+    <!-- tail -->
+    <visual>
+      <origin xyz="${-(body_length/2 + tail_length/2)} 0 ${(body_height - head_height)/2}" rpy="0 0 0"/>
+      <geometry><box size="${tail_length} ${head_width} ${head_height}"/></geometry>
+      <material name="dark_grey"/>
+    </visual>
   </link>
-  <!-- IMU link (center of body) -->
+  <!-- base_footprint: base_link projected onto the ground (REP-105) -->
+  <joint name="base_footprint_joint" type="fixed">
+    <parent link="base_link"/>
+    <child  link="base_footprint"/>
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